File: power-ice.kicad_pcb (KiCad board)
At the start: 2 copper layers, 92.1 x 51.4 mm, 63 parts, among them J1 Conn_01x03_Female, J2 Conn_01x02_Female, J3 Conn_01x02_Female, U1 LM318N, U2 LM318N, U3 LM318N, U4 LM318N, U5 LM318N, U6 LM318N, U7 LM318N

Commit message: redesign
Parts:
- removed the C14 at (152.2, 92.1)
- removed C19, C20: C, Capacitor_SMD:C_0805_2012Metric_Pad1.15x1.40mm_HandSolder
- removed C21: 100n, Capacitor_SMD:C_0805_2012Metric_Pad1.15x1.40mm_HandSolder
- removed C22: 1n, Capacitor_SMD:C_1206_3216Metric_Pad1.42x1.75mm_HandSolder
- removed JP1, JP2, JP3, JP4, JP5: Jumper, Jumper:SolderJumper-2_P1.3mm_Open_Pad1.0x1.5mm
- removed U6, U7: LM318N, Package_DIP:DIP-8_W7.62mm
- added C14: C, Capacitor_SMD:C_0805_2012Metric, F.Cu at (112.3, 58.1)
- added C14: C, Capacitor_SMD:C_0805_2012Metric, F.Cu at (102.6, 79.7)
- added D4: LED, LED_THT:LED_D2.0mm_W4.0mm_H2.8mm_FlatTop, F.Cu at (123.8, 31.3)
- added D5: D_Photo, Connector_PinHeader_2.54mm:PinHeader_1x02_P2.54mm_Vertical, F.Cu at (125.2, 38.9)
- added D6: LED, LED_THT:LED_D2.0mm_W4.0mm_H2.8mm_FlatTop, F.Cu at (116.2, 44.5)
- added D7: LED, LED_THT:LED_D2.0mm_W4.0mm_H2.8mm_FlatTop, F.Cu at (131.6, 34.9)
- added J4: Conn_01x01_Female, Connector_PinHeader_2.54mm:PinHeader_1x01_P2.54mm_Vertical, F.Cu at (120.2, 61.7)
- added J5: Conn_01x01_Female, Connector_PinHeader_2.54mm:PinHeader_1x01_P2.54mm_Vertical, F.Cu at (120.0, 77.1)
- added Q1: Q_NMOS_DGS, Package_TO_SOT_THT:TO-220-3_Vertical, F.Cu at (146.0, 45.4)
- added Q2: Q_NMOS_DGS, Package_TO_SOT_THT:TO-220-3_Vertical, F.Cu at (146.7, 30.2)
- added Q3: Q_NMOS_DGS, Package_TO_SOT_THT:TO-220-3_Vertical, F.Cu at (184.1, 44.7)
- added Q4: Q_NMOS_DGS, Package_TO_SOT_THT:TO-220-3_Vertical, F.Cu at (184.8, 30.6)
- added Q5: Q_NMOS_DGS, Package_TO_SOT_THT:TO-220-3_Vertical, F.Cu at (165.2, 44.1)
- added Q6: Q_NMOS_DGS, Package_TO_SOT_THT:TO-220-3_Vertical, F.Cu at (165.7, 30.6)
- added R24: 18k, Resistor_SMD:R_0805_2012Metric, F.Cu at (161.9, 59.4)
- added R25: 10k, Resistor_SMD:R_0805_2012Metric, F.Cu at (162.9, 62.4)
- added R26: 15, Resistor_THT:R_Axial_DIN0204_L3.6mm_D1.6mm_P1.90mm_Vertical, F.Cu at (174.4, 44.3)
- added R27: 18k, Resistor_SMD:R_0805_2012Metric, F.Cu at (172.0, 64.9)
- added R28: 10k, Resistor_SMD:R_0805_2012Metric, F.Cu at (172.9, 67.9)
- added R29: 15, Resistor_THT:R_Axial_DIN0204_L3.6mm_D1.6mm_P1.90mm_Vertical, F.Cu at (175.0, 30.6)
- C1, C2: value 220u -> C; footprint Capacitor_THT:C_Disc_D11.0mm_W5.0mm_P7.50mm -> Capacitor_SMD:C_0805_2012Metric
- C10, C12, C4, C6, C8: value 1n -> C; footprint Capacitor_SMD:C_1206_3216Metric_Pad1.42x1.75mm_HandSolder -> Capacitor_SMD:C_0805_2012Metric
- C11, C13, C3, C5, C7, C9: value 100n -> C; footprint Capacitor_SMD:C_0805_2012Metric_Pad1.15x1.40mm_HandSolder -> Capacitor_SMD:C_0805_2012Metric
- C15, C16, C17, C18: footprint Capacitor_SMD:C_0805_2012Metric_Pad1.15x1.40mm_HandSolder -> Capacitor_SMD:C_0805_2012Metric
- D1: value D_Photo -> LED; footprint Connector_PinHeader_2.54mm:PinHeader_2x01_P2.54mm_Vertical -> LED_THT:LED_D2.0mm_W4.0mm_H2.8mm_FlatTop
- D2: value D_Schottky -> LED; footprint Connector_PinHeader_2.54mm:PinHeader_2x01_P2.54mm_Vertical -> LED_THT:LED_D2.0mm_W4.0mm_H2.8mm_FlatTop
- D3: value 3.3V -> LED; footprint Connector_PinHeader_2.54mm:PinHeader_2x01_P2.54mm_Vertical -> LED_THT:LED_D2.0mm_W4.0mm_H2.8mm_FlatTop
- J1: value Conn_01x03_Female -> Conn_01x07_Female; footprint Connector_PinHeader_2.54mm:PinHeader_1x03_P2.54mm_Vertical -> Connector_PinSocket_2.54mm:PinSocket_1x07_P2.54mm_Vertical
- J2: value Conn_01x02_Female -> Conn_01x03_Female; footprint Connector_PinSocket_2.54mm:PinSocket_1x02_P2.54mm_Vertical -> Connector_PinSocket_2.54mm:PinSocket_1x03_P2.54mm_Vertical
- J3: value Conn_01x02_Female -> Conn_01x01_Female; footprint Connector_PinSocket_2.54mm:PinSocket_1x02_P2.54mm_Vertical -> Connector_Wire:SolderWire-2.5sqmm_1x01_D2.4mm_OD3.6mm
- R1, R10: value 1k -> 18k; footprint Resistor_SMD:R_0805_2012Metric_Pad1.15x1.40mm_HandSolder -> Resistor_SMD:R_0805_2012Metric
- R11, R18, R19, R2, R20, R21, R22, R23, R5: footprint Resistor_SMD:R_0805_2012Metric_Pad1.15x1.40mm_HandSolder -> Resistor_SMD:R_0805_2012Metric
- R12, R6: value 1k -> 15; footprint Resistor_SMD:R_0805_2012Metric_Pad1.15x1.40mm_HandSolder -> Resistor_THT:R_Axial_DIN0204_L3.6mm_D1.6mm_P1.90mm_Vertical
- R13, R15, R17: value 10k -> R; footprint Resistor_SMD:R_0805_2012Metric_Pad1.15x1.40mm_HandSolder -> Resistor_SMD:R_0805_2012Metric
- R14: value 22k -> R; footprint Resistor_SMD:R_0805_2012Metric_Pad1.15x1.40mm_HandSolder -> Resistor_SMD:R_0805_2012Metric
- R16: value 1k -> R; footprint Resistor_SMD:R_0805_2012Metric_Pad1.15x1.40mm_HandSolder -> Resistor_SMD:R_0805_2012Metric
- R3: value 4.7k -> 15; footprint Resistor_SMD:R_0805_2012Metric_Pad1.15x1.40mm_HandSolder -> Resistor_THT:R_Axial_DIN0204_L3.6mm_D1.6mm_P1.90mm_Vertical
- R4: value 4.7k -> 18k; footprint Resistor_SMD:R_0805_2012Metric_Pad1.15x1.40mm_HandSolder -> Resistor_SMD:R_0805_2012Metric
- R7: value 10k -> 18k; footprint Resistor_SMD:R_0805_2012Metric_Pad1.15x1.40mm_HandSolder -> Resistor_SMD:R_0805_2012Metric
- R8: value 1k -> 10k; footprint Resistor_SMD:R_0805_2012Metric_Pad1.15x1.40mm_HandSolder -> Resistor_SMD:R_0805_2012Metric
- R9: value 10k -> 15; footprint Resistor_SMD:R_0805_2012Metric_Pad1.15x1.40mm_HandSolder -> Resistor_THT:R_Axial_DIN0204_L3.6mm_D1.6mm_P1.90mm_Vertical
- U1, U2, U3, U4, U5: value LM318N -> MCP6002-xP
- moved U2 97.9 mm to (186.7, 56.7)
- moved R3 89.6 mm to (155.6, 45.0), turned to 0 degrees
- moved R12 89.2 mm to (194.2, 30.6), turned to 0 degrees
- moved R4 79.4 mm to (152.3, 65.8), turned to -90 degrees
- moved J1 72.0 mm to (145.1, 79.2), turned to 90 degrees
- moved C8 69.2 mm to (197.9, 53.5), turned to 0 degrees
- moved C7 67.9 mm to (197.9, 55.7), turned to 0 degrees
- moved C2 67.7 mm to (102.3, 29.1), turned to 90 degrees
- moved C1 63.3 mm to (104.7, 29.1), turned to -90 degrees
- moved C13 61.5 mm to (107.8, 46.9)
- moved D1 60.1 mm to (132.1, 46.3), turned to 45 degrees
- moved R5 56.6 mm to (148.9, 65.1), turned to 0 degrees
- moved J2 55.7 mm to (99.4, 27.8)
- moved R11 55.3 mm to (197.3, 67.2), turned to 180 degrees
- moved R10 53.2 mm to (193.2, 67.2)
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Connections:
- C1 pad 1: +10V -> GND
- C1 pad 2: GND -> +3V3
- C10 pad 1: +10V -> +3V3
- C10 pad 2: -10V -> GNDA
- C11 pad 1: +10V -> +3V3
- C11 pad 2: -10V -> GNDA
- C12 pad 1: +10V -> Net-(C12-Pad1)
- C12 pad 2: -10V -> Net-(C12-Pad2)
- C13 pad 1: +10V -> +3V3
- C13 pad 2: -10V -> GNDA
- C15 pad 1: /cascade_filter/out -> Net-(C15-Pad1)
- C15 pad 2: GND -> Net-(C15-Pad2)
- C16 pad 1: /sheet6215D380/out -> Net-(C16-Pad1)
- C16 pad 2: GND -> GNDA
- C17 pad 1: /sheet62163674/out -> +5V
- C18 pad 1: /sheet621688F6/out -> +5V
- C2 pad 1: GND -> +3V3
- C2 pad 2: -10V -> GND
- C3 pad 1: +10V -> +5V
- C3 pad 2: -10V -> GND
- C4 pad 1: +10V -> +5V
- C4 pad 2: -10V -> GND
- C5 pad 1: +10V -> +5V
- C5 pad 2: -10V -> GND
- C6 pad 1: +10V -> +5V
- C6 pad 2: -10V -> GND
- C7 pad 1: +10V -> +5V
- C7 pad 2: -10V -> GND
- C8 pad 1: +10V -> +5V
- C8 pad 2: -10V -> GND
- C9 pad 1: +10V -> +3V3
- C9 pad 2: -10V -> GNDA
- D1 pad 2: GND -> +5V
- D2 pad 2: amp_out -> +5V
- D3 pad 2: GND -> +5V
- J1 pad 1: GND -> /IR_LED/InputLedAblock
- J1 pad 2: -10V -> /IR_LED/InputLedBblock
- J1 pad 3: +10V -> /sheet6238A8B8/InputLedAblock
- J2 pad 1: -10V -> GND
- J2 pad 2: +10V -> +3V3
- J3 pad 1: Net-(D3-Pad1) -> GNDA
- R1 pad 2: /sheet6216EEAD/in -> /IR_LED/InputLedAblock
- R10 pad 2: /sheet6215D380/in -> /sheet62353F20/InputLedBblock
- R11 pad 1: /sheet6215D380/in -> GND
- R11 pad 2: GND -> Net-(R10-Pad1)
- R12 pad 1: Net-(R12-Pad1) -> Net-(Q4-Pad3)
- R12 pad 2: /cascade_filter/in -> GND
- R13 pad 1: /cascade_filter/in -> Net-(R13-Pad1)
- R13 pad 2: GND -> Net-(D5-Pad1)
- R14 pad 1: Net-(D3-Pad1) -> Net-(R14-Pad1)
- R14 pad 2: Net-(D2-Pad1) -> GNDA
- R15 pad 1: GND -> Net-(C12-Pad2)
- R15 pad 2: Net-(D3-Pad1) -> Net-(R14-Pad1)
- R16 pad 1: Net-(R16-Pad1) -> Net-(C12-Pad1)
- R16 pad 2: /sheet62181AF4/in -> GNDA
- R17 pad 1: /sheet62181AF4/in -> Net-(C14-Pad1)
- R17 pad 2: GND -> Net-(C12-Pad1)
- R18 pad 1: /cascade_filter/in -> Net-(R18-Pad1)
- R18 pad 2: /cascade_filter/out -> GNDA
- R19 pad 1: /sheet6215D380/in -> Net-(C15-Pad2)
- R19 pad 2: /sheet6215D380/out -> Net-(R18-Pad1)
- R2 pad 1: /sheet6216EEAD/in -> GND
- R2 pad 2: GND -> Net-(R1-Pad1)
- R20 pad 1: /sheet62163674/in -> Net-(C15-Pad1)
- R20 pad 2: /sheet62163674/out -> GNDA
- R21 pad 1: /sheet621688F6/in -> Net-(C16-Pad1)
- R21 pad 2: /sheet621688F6/out -> Net-(C15-Pad1)
- R22 pad 1: /sheet6216EEAD/in -> Net-(R22-Pad1)
- R22 pad 2: /sheet6216EEAD/out -> GNDA
- R23 pad 1: /sheet62181AF4/in -> /Sheet6239F98A/OutputPDCircuit
- R23 pad 2: amp_out -> Net-(R22-Pad1)
- R3 pad 1: +10V -> Net-(Q1-Pad3)
- R4 pad 1: GND -> Net-(R4-Pad1)
- R4 pad 2: -10V -> /IR_LED/InputLedBblock
- R5 pad 1: op_cascade_in -> GND
- R5 pad 2: Net-(D1-Pad1) -> Net-(R4-Pad1)
- R6 pad 1: Net-(R6-Pad1) -> Net-(Q2-Pad3)
- R6 pad 2: /sheet621688F6/in -> GND
- R7 pad 1: /sheet621688F6/in -> Net-(R7-Pad1)
- R7 pad 2: GND -> /sheet62353F20/InputLedAblock
- R8 pad 1: Net-(R8-Pad1) -> GND
- R8 pad 2: /sheet62163674/in -> Net-(R7-Pad1)
- R9 pad 1: /sheet62163674/in -> Net-(Q3-Pad3)
- U1 pad 2: Net-(R1-Pad1) -> Net-(Q1-Pad3)
- U1 pad 3: op_cascade_in -> Net-(R1-Pad1)
- U1 pad 4: -10V -> GND
- U1 pad 5: Net-(U1-Pad5) -> Net-(R4-Pad1)
- U1 pad 6: /sheet6216EEAD/in -> Net-(Q2-Pad3)
- U1 pad 7: +10V -> Net-(Q2-Pad2)
- U1 pad 8: Net-(U1-Pad8) -> unconnected-(U1-Pad8)
- U2 pad 2: Net-(D1-Pad1) -> Net-(Q3-Pad3)
- U2 pad 3: GND -> Net-(R7-Pad1)
- U2 pad 4: -10V -> GND
- U2 pad 5: Net-(U2-Pad5) -> Net-(R10-Pad1)
- U2 pad 6: op_cascade_in -> Net-(Q4-Pad3)
- U2 pad 7: +10V -> Net-(Q4-Pad2)
- U2 pad 8: Net-(U2-Pad8) -> unconnected-(U2-Pad8)
- U3 pad 1: Net-(U3-Pad1) -> Net-(R13-Pad1)
- U3 pad 2: Net-(R6-Pad1) -> Net-(D5-Pad1)
- U3 pad 3: /sheet6216EEAD/out -> GNDA
- U3 pad 4: -10V -> GNDA
- U3 pad 5: Net-(U3-Pad5) -> Net-(R13-Pad1)
- U3 pad 6: /sheet621688F6/in -> Net-(R14-Pad1)
- U3 pad 7: +10V -> Net-(C12-Pad2)
- U3 pad 8: Net-(U3-Pad8) -> +3V3
- U4 pad 1: Net-(U4-Pad1) -> Net-(C15-Pad2)
- U4 pad 2: Net-(R8-Pad1) -> Net-(R18-Pad1)
- U4 pad 3: /sheet621688F6/out -> Net-(C14-Pad1)
- U4 pad 4: -10V -> GNDA
- U4 pad 5: Net-(U4-Pad5) -> Net-(C16-Pad1)
- U4 pad 6: /sheet62163674/in -> Net-(R22-Pad1)
- U4 pad 7: +10V -> /Sheet6239F98A/OutputPDCircuit
- U4 pad 8: Net-(U4-Pad8) -> +3V3
- U5 pad 2: Net-(R10-Pad1) -> Net-(Q5-Pad3)
- U5 pad 3: /sheet62163674/out -> Net-(R24-Pad1)
- U5 pad 4: -10V -> GND
- U5 pad 6: /sheet6215D380/in -> Net-(Q6-Pad3)
- U5 pad 7: +10V -> Net-(Q6-Pad2)
- U5 pad 8: Net-(U5-Pad8) -> unconnected-(U5-Pad8)
Routing:
- net +5V: track 0.00 -> 170.0 mm
- net Net-(D3-Pad1): track 0.00 -> 86.2 mm
- net /Sheet6239F98A/OutputPDCircuit: track 0.00 -> 70.0 mm
- net Net-(D4-Pad1): track 0.00 -> 67.1 mm
- net +3V3: track 0.00 -> 63.6 mm
- net Net-(D5-Pad1): track 0.00 -> 61.1 mm
- net Net-(D6-Pad1): track 0.00 -> 51.5 mm
- net Net-(Q4-Pad3): track 0.00 -> 46.4 mm
- net Net-(Q6-Pad3): track 0.00 -> 44.0 mm
- net Net-(C14-Pad1): track 0.00 -> 43.8 mm
- net Net-(Q2-Pad3): track 0.00 -> 42.2 mm
- net /sheet62353F20/InputLedBblock: track 0.00 -> 40.7 mm
- net Net-(Q6-Pad2): track 0.00 -> 38.8 mm
- net /sheet62353F20/InputLedAblock: track 0.00 -> 38.7 mm
- net Net-(Q2-Pad2): track 0.00 -> 35.9 mm
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- added copper zone on B.Cu, net GNDA
- added copper zone on F.Cu, net GNDA
Other:
- board size 92.1 x 51.4 mm -> 115 x 57 mm
- net class Default removed
- board text added: "LED"
