File: power-ice.sch (KiCad schematic (older format))
At the start: 51 parts, among them J1 Conn_01x03_Female, J2 Conn_01x02_Female, J3 Conn_01x02_Female, U1 LM318N, U2 LM318N, U3 LM318N, U4 LM318N, U5 LM318N, U6 LM318N, U7 LM318N

Commit message: redesign
Parts:
- removed C1, C2: 220u, Capacitor_THT:C_Disc_D11.0mm_W5.0mm_P7.50mm, symbol Device:C
- removed C10, C12, C14, C22, C4, C6, C8: 1n, Capacitor_SMD:C_1206_3216Metric_Pad1.42x1.75mm_HandSolder, symbol Device:C
- removed C11, C13, C21, C3, C5, C7, C9: 100n, Capacitor_SMD:C_0805_2012Metric_Pad1.15x1.40mm_HandSolder, symbol Device:C
- removed D1: D_Photo, Connector_PinHeader_2.54mm:PinHeader_2x01_P2.54mm_Vertical, symbol Device:D_Photo
- removed D2: D_Schottky, Connector_PinHeader_2.54mm:PinHeader_2x01_P2.54mm_Vertical, symbol Device:D_Schottky
- removed D3: 3.3V, Connector_PinHeader_2.54mm:PinHeader_2x01_P2.54mm_Vertical, symbol Device:D_Zener
- removed J1: Conn_01x03_Female, Connector_PinHeader_2.54mm:PinHeader_1x03_P2.54mm_Vertical, symbol Connector:Conn_01x03_Female
- removed J2, J3: Conn_01x02_Female, Connector_PinSocket_2.54mm:PinSocket_1x02_P2.54mm_Vertical, symbol Connector:Conn_01x02_Female
- removed JP1, JP2, JP3, JP4, JP5: Jumper, Jumper:SolderJumper-2_P1.3mm_Open_Pad1.0x1.5mm, symbol Device:Jumper
- removed R1, R10, R12, R16, R6, R8: 1k, Resistor_SMD:R_0805_2012Metric_Pad1.15x1.40mm_HandSolder, symbol Device:R
- removed R11, R13, R15, R17, R2, R5, R7, R9: 10k, Resistor_SMD:R_0805_2012Metric_Pad1.15x1.40mm_HandSolder, symbol Device:R
- removed R14: 22k, Resistor_SMD:R_0805_2012Metric_Pad1.15x1.40mm_HandSolder, symbol Device:R
- removed R3, R4: 4.7k, Resistor_SMD:R_0805_2012Metric_Pad1.15x1.40mm_HandSolder, symbol Device:R
- removed U1, U2, U3, U4, U5, U6, U7: LM318N, Package_DIP:DIP-8_W7.62mm, symbol Amplifier_Operational:LM318N
- added C15, C16, C17, C18: C, Capacitor_SMD:C_0805_2012Metric, symbol pspice:C
- added J1: Conn_01x13_Female, Connector_PinSocket_2.54mm:PinSocket_1x13_P2.54mm_Horizontal, symbol Connector:Conn_01x13_Female
- added J2: Conn_01x03_Female, Connector_PinSocket_2.54mm:PinSocket_1x03_P2.54mm_Vertical, symbol Connector:Conn_01x03_Female
Connections:
- net labels added: +3.3V, +5V
- net labels removed: +10V, +24V, -10V, GNDPWR, amp_out, op_cascade_in
- wire segments 117 -> 66
- no-connect marks 21 -> 0
